Commit message: depth_map and disparity_image obtained but some inaccuracy in depth_est and stereo_camera_plugins added to both quadruped and husky

File: simulator/urdf/component_snippets.xacro (robot description, xacro)
@@ -2,5 +2,98 @@
 <robot xmlns:xacro="http://ros.org/wiki/xacro">
     <xacro:property name="pi" value="3.14159265359" />
-    <xacro:macro name="camera_macro"
+    <xacro:macro name="stereocamera_macro"
+    params="namespace parent_link camera_suffix frame_rate
+      horizontal_fov image_width image_height image_format min_distance
+      max_distance noise_mean noise_stddev enable_visual *geometry *origin">
+    <link name="${namespace}/stereocamera_${camera_suffix}_link">
+      <collision>
+        <origin xyz="0 0 0" rpy="0 0 0" />
+        <geometry>
+          <xacro:insert_block name="geometry" />
+        </geometry>
+      </collision>
+      <xacro:if value="${enable_visual}">
+        <visual>
+          <origin xyz="0 0 0" rpy="0 ${pi/2} 0" />
+          <geometry>
+            <xacro:insert_block name="geometry" />
+          </geometry>
+          <material name="red" />
+        </visual>
+      </xacro:if>
+      <inertial>
+        <mass value="1e-5" />
+        <origin xyz="0 0 0" rpy="0 0 0" />
+        <inertia ixx="1e-6" ixy="0" ixz="0" iyy="1e-6" iyz="0" izz="1e-6" />
+      </inertial>
+    </link>
+    <joint name="${namespace}/stereocamera_${camera_suffix}_joint" type="fixed">
+      <xacro:insert_block name="origin" />
+      <parent link="${parent_link}" />
+      <child link="${namespace}/stereocamera_${camera_suffix}_link" />
+    </joint>
+    <link name="${namespace}/stereocamera_${camera_suffix}_optical_link" />
+    <joint name="${namespace}/stereocamera_${camera_suffix}_optical_joint" type="fixed" >
+      <origin xyz="0 0 0" rpy="${-pi/2} 0 ${-pi/2}" />
+      <parent link="${namespace}/stereocamera_${camera_suffix}_link" />
+      <child link="${namespace}/stereocamera_${camera_suffix}_optical_link" />
+    </joint>
+    <gazebo reference="${namespace}/stereocamera_${camera_suffix}_link">
+      <sensor type="multicamera" name="stereo_camera">
+        <update_rate>${frame_rate}</update_rate>
+        <camera name="left">
+          <horizontal_fov>${horizontal_fov}</horizontal_fov>
+          <image>
+            <width>${image_width}</width>
+            <height>${image_height}</height>
+            <format>${image_format}</format>
+          </image>
+          <clip>
+            <near>${min_distance}</near>
+            <far>${max_distance}</far>
+          </clip>
+          <noise>
+            <type>gaussian</type>
+            <mean>${noise_mean}</mean>
+            <stddev>${noise_stddev}</stddev>
+          </noise>
+        </camera>
+        <camera name="right">
+        <pose>0 -0.07 0 0 0 0</pose>
+        <horizontal_fov>${horizontal_fov}</horizontal_fov>
+          <image>
+            <width>${image_width}</width>
+            <height>${image_height}</height>
+            <format>${image_format}</format>
+          </image>
+          <clip>
+            <near>${min_distance}</near>
+            <far>${max_distance}</far>
+          </clip>
+          <noise>
+            <type>gaussian</type>
+            <mean>${noise_mean}</mean>
+            <stddev>${noise_stddev}</stddev>
+          </noise>
+        </camera>
+        <plugin name="stereo_camera_controller" filename="libgazebo_ros_multicamera.so">
+          <robotNamespace>${namespace}</robotNamespace>
+          <alwaysOn>true</alwaysOn>
+          <updateRate>${frame_rate}</updateRate>
+          <cameraName>stereocamera_${camera_suffix}</cameraName>
+          <imageTopicName>image_raw</imageTopicName>
+          <cameraInfoTopicName>camera_info</cameraInfoTopicName>
+          <frameName>camera_${camera_suffix}_link</frameName>
+          <hackBaseline>0.07</hackBaseline>
+          <distortionK1>0.0</distortionK1>
+          <distortionK2>0.0</distortionK2>
+          <distortionK3>0.0</distortionK3>
+          <distortionT1>0.0</distortionT1>
+          <distortionT2>0.0</distortionT2>
+        </plugin>
+      </sensor>
+    </gazebo>
+    </xacro:macro>
+    <!--<xacro:macro name="camera_macro"
     params="namespace parent_link camera_suffix frame_rate
       horizontal_fov image_width image_height image_format min_distance
@@ -55,7 +148,4 @@
           <noise>
             <type>gaussian</type>
-            <!-- Noise is sampled independently per pixel on each frame.
-                 That pixel's noise value is added to each of its color
-                 channels, which at that point lie in the range [0,1]. -->
             <mean>${noise_mean}</mean>
             <stddev>${noise_stddev}</stddev>
@@ -171,9 +261,9 @@
           <noise>
             <type>gaussian</type>
-            <!-- Noise parameters based on published spec for Hokuyo laser
+            --><!-- Noise parameters based on published spec for Hokuyo laser
                  achieving "+-30mm" accuracy at range < 10m.  A mean of 0.0m and
                  stddev of 0.01m will put 99.7% of samples within 0.03m of the true
                  reading. -->
-            <mean>0.0</mean>
+           <!-- <mean>0.0</mean>
             <stddev>0.01</stddev>
           </noise>
@@ -189,4 +279,4 @@
       <disableFixedJointLumping>true</disableFixedJointLumping>
     </gazebo>
-    </xacro:macro>
+    </xacro:macro>-->
 </robot>

File: simulator/urdf/quadruped_base.xacro (robot description, xacro)
@@ -2,5 +2,23 @@
 <robot name="$(arg ugv_name)" xmlns:xacro="http://ros.org/wiki/xacro">
     <xacro:include filename="$(find simulator)/urdf/component_snippets.xacro" />
-    <!-- Instantiate firefly "mechanics" -->
+    <xacro:include filename="$(find simulator)/urdf/quadruped.xacro" />
+    <xacro:stereocamera_macro
+    namespace=""
+    parent_link="base_link"
+    camera_suffix="front"
+    frame_rate="30"
+    horizontal_fov="1.57"
+    image_width="640"
+    image_height="480"
+    image_format="R8G8B8"
+    min_distance="0.02"
+    max_distance="300"
+    noise_mean="0.0"
+    noise_stddev="0.007"
+    enable_visual="true">
+    <box size="0.02 0.02 0.02"/>
+    <origin xyz="0.14 0.0 0.02" rpy="0.0 0.0 0.0" />
+    </xacro:stereocamera_macro>
+    <!-- Instantiate firefly "mechanics"
     <xacro:include filename="$(find simulator)/urdf/quadruped.xacro" />
     <xacro:camera_macro
@@ -65,4 +83,4 @@
     lidar_topic="lidar/right">
     <origin xyz="0.0 -0.14 -0.02" rpy="0.0 0.0 -1.57"/>
-    </xacro:lidar_macro>
+    </xacro:lidar_macro>-->
 </robot>
